File: Sequencer/Sequencer.kicad_sch (KiCad schematic)
At the start: 67 parts, among them J6 EURO_PWR_2x5, SW4 SW_8/16, U1 MCP23017_SP, U2 TL084, U3 L7805

Commit message: Sequencer progress
Parts:
- removed C6, C8: 100n, Capacitor_THT:C_Disc_D4.7mm_W2.5mm_P5.00mm, symbol Device:C
- removed J6: EURO_PWR_2x5, Connector_PinHeader_2.54mm:PinHeader_2x05_P2.54mm_Vertical, symbol eurocad:EURO_PWR_2x5
- removed R1, R10, R11, R12, R13, R14, R15, R16, R2, R3, R4, R5, R6, R7, R8, R9: 100K, Resistor_THT:R_Axial_DIN0207_L6.3mm_D2.5mm_P2.54mm_Vertical, symbol Device:R
- removed U2: TL084, Package_DIP:DIP-14_W7.62mm_Socket, symbol Amplifier_Operational:TL084
- added D1, D11, D12, D15, D16, D17, D18, D2, D21, D22, D23, D24, D5, D6, D7, D8: 1N4148, Diode_THT:D_DO-35_SOD27_P7.62mm_Horizontal, symbol Diode:1N4148
- added J1: Power, Connector_PinHeader_2.54mm:PinHeader_2x05_P2.54mm_Vertical, symbol Connector_Generic:Conn_02x05_Odd_Even
- RV1, RV16: value A10K -> B10K
- RV10: renamed from RV13; value A10K -> B10K
- RV11: renamed from RV6; value A10K -> B10K
- RV12: renamed from RV14; value A10K -> B10K
- RV13: renamed from RV7; value A10K -> B10K
- RV14: renamed from RV15; value A10K -> B10K
- RV15: renamed from RV8; value A10K -> B10K
- RV2: renamed from RV9; value A10K -> B10K
- RV3: renamed from RV2; value A10K -> B10K
- RV4: renamed from RV10; value A10K -> B10K
- RV5: renamed from RV3; value A10K -> B10K
- RV6: renamed from RV11; value A10K -> B10K
- RV7: renamed from RV4; value A10K -> B10K
- RV8: renamed from RV12; value A10K -> B10K
- RV9: renamed from RV5; value A10K -> B10K
- renumbered C7 to C1, C4 to C2, C5 to C3, D6 to D10, D3 to D13, D7 to D14, D4 to D19, D8 to D20, D1 to D3, D5 to D4, D2 to D9, R17 to R1, R22 to R10, R29 to R11, R30 to R12, R23 to R13, R24 to R14, R31 to R15, R32 to R16, R18 to R2, R25 to R3, R26 to R4, R19 to R5, R20 to R6, R27 to R7, R28 to R8, R21 to R9, SW4 to SW1, U3 to U2
Connections:
- net +12V: now also J1.10 (Pin_10), J1.9 (Pin_9)
- net -12V: now also J1.1 (Pin_1), J1.2 (Pin_2)
- net CV1_OUT: now also D1.1 (K), D11.1 (K), D15.1 (K), D17.1 (K), D21.1 (K), D23.1 (K), D5.1 (K), D7.1 (K)
- net GND: now also J1.3 (Pin_3), J1.4 (Pin_4), J1.5 (Pin_5), J1.6 (Pin_6), J1.7 (Pin_7), J1.8 (Pin_8)
- net STEP10: now also U1.27 (GPA6); no longer U1.22 (GPA1)
- net STEP11: now also U1.26 (GPA5); no longer U1.23 (GPA2)
- net STEP12: now also U1.25 (GPA4); no longer U1.24 (GPA3)
- net STEP13: now also U1.24 (GPA3); no longer U1.25 (GPA4)
- net STEP14: now also U1.23 (GPA2); no longer U1.26 (GPA5)
- net STEP15: now also U1.22 (GPA1); no longer U1.27 (GPA6)
- net STEP16: now also U1.21 (GPA0); no longer U1.28 (GPA7)
- net STEP9: now also U1.28 (GPA7); no longer U1.21 (GPA0)
- net at RV12.2: now also D18.2 (A)
- net at SW1.5 (B): now also D12.1 (K), D16.1 (K), D18.1 (K), D2.1 (K), D22.1 (K), D24.1 (K), D6.1 (K), D8.1 (K)
- net at RV5.2: now also D7.2 (A)
- net at RV6.2: now also D8.2 (A)
- net at RV15.2: now also D23.2 (A)
- net at RV8.2: now also D12.2 (A)
- net at RV13.2: now also D21.2 (A)
- net at RV1.2: now also D1.2 (A)
- net at RV9.2: now also D15.2 (A)
- net at RV11.2: now also D17.2 (A)
- net at RV14.2: now also D22.2 (A)
- net at RV16.2: now also D24.2 (A)
- net at RV10.2: now also D16.2 (A)
- net at RV3.2: now also D5.2 (A)
- net at RV4.2: now also D6.2 (A)
- net at RV2.2: now also D2.2 (A)
- net at RV7.2: now also D11.2 (A)
- net CLOCK_IN renamed STEP_IN
Other:
- moved on the sheet: C1, C2, C3, RV1, RV10, RV11, RV12, RV13, RV14, RV15, RV16, RV2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

Commit message: Sequencer Progress
Parts:
- removed J1: Power, Connector_PinHeader_2.54mm:PinHeader_2x05_P2.54mm_Vertical, symbol Connector_Generic:Conn_02x05_Odd_Even
Other:
- sheet INPUTSOUTPUTS renamed FRONTEND
- moved on the sheet: C1, C2, C3, SW1A, U2
