File: Sequencer/inputs.kicad_sch (KiCad schematic)
At the start: 50 parts, among them J1 CLOCK_IN, J2 RESET_IN, J3 FLIP_IN, J4 CV1_OUT, J5 CV2_OUT, Q1 2N3904, Q2 2N3904, Q3 2N3904, SW1 SW_STEP, SW2 SW_RESET, SW3 SW_FLIP, U2 TL084

Commit message: Sequencer progress
Parts:
- removed R52, R53, R59, R60: 10K, Resistor_THT:R_Axial_DIN0207_L6.3mm_D2.5mm_P2.54mm_Vertical, symbol Device:R
- removed R55: 68K, Resistor_THT:R_Axial_DIN0207_L6.3mm_D2.5mm_P2.54mm_Vertical, symbol Device:R
- removed R56: 18K, Resistor_THT:R_Axial_DIN0207_L6.3mm_D2.5mm_P2.54mm_Vertical, symbol Device:R
- removed R57: 100K, Resistor_THT:R_Axial_DIN0207_L6.3mm_D2.5mm_P2.54mm_Vertical, symbol Device:R
- removed R58: 220K, Resistor_THT:R_Axial_DIN0207_L6.3mm_D2.5mm_P2.54mm_Vertical, symbol Device:R
- removed R61: 1K, Resistor_THT:R_Axial_DIN0207_L6.3mm_D2.5mm_P2.54mm_Vertical, symbol Device:R
- removed U2: TL084, Package_DIP:DIP-14_W7.62mm_Socket, symbol Amplifier_Operational:TL084
- added C7, C8: 100n, Capacitor_THT:C_Disc_D4.7mm_W2.5mm_P5.00mm, symbol Device:C
- added R35, R37: 3k3, Resistor_THT:R_Axial_DIN0207_L6.3mm_D2.5mm_P2.54mm_Vertical, symbol Device:R
- added R36, R38, R39: 10k, Resistor_THT:R_Axial_DIN0207_L6.3mm_D2.5mm_P2.54mm_Vertical, symbol Device:R
- added R41: 33k, Resistor_THT:R_Axial_DIN0207_L6.3mm_D2.5mm_P2.54mm_Vertical, symbol Device:R
- added R43: 1K, Resistor_THT:R_Axial_DIN0207_L6.3mm_D2.5mm_P2.54mm_Vertical, symbol Device:R
- added U3: TL082, symbol Amplifier_Operational:TL082
- R32: renamed from R48; value 68K -> 10K
- R33: renamed from R49; value 18K -> 10K
- R34: renamed from R50; value 100K -> 10k
- R40: renamed from R51; value 220K -> 33k
- renumbered C1 to C4, C2 to C5, C3 to C6, D9 to D25, D10 to D26, D13 to D27, D11 to D28, D12 to D29, D14 to D30, J1 to J2, J2 to J3, J3 to J4, J4 to J5, J5 to J6, R33 to R17, R34 to R18, R43 to R19, R35 to R20, R36 to R21, R44 to R22, R37 to R23, R38 to R24, R45 to R25, R39 to R26, R40 to R27, R46 to R28, R41 to R29, R42 to R30, R47 to R31, R54 to R42, SW1 to SW2, SW2 to SW3, SW3 to SW4
Connections:
- net +5V: now also R32.1
- net -12V: now also C8.2, U3.4 (V-); no longer R32.1
- net CV1_OUT: now also R35.2; no longer R34.2, R40.1
- net CV2_OUT: now also R37.2
- net GND: now also C7.2, C8.1, R38.1, R39.1
- net at R32.2, R33.1, R34.1: now also R36.1
- net at R40.2: now also R42.1, U3.1
- net at J6.3: now also R43.2
- net CLOCK_IN renamed STEP_IN
- new net: R36.2, R41.1, U3.6 (-)
- new net: R34.2, R40.1, U3.2 (-)
- new net: R35.1, R38.2, U3.3 (+)
- new net: R37.1, R39.2, U3.5 (+)
- new net: R41.2, R43.1, U3.7
- new net +12V: C7.1, U3.8 (V+)
Other:
- note added: "-8..8v"
- note added: "0..5v"
- note added: "2.5v"
- moved on the sheet: C4, C5, C6, D25, D26, D27, D28, D29, D30, J2, J3, J4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

Commit message: Sequencer Progress
Parts:
- added J1: Power, Connector_PinHeader_2.54mm:PinHeader_2x05_P2.54mm_Vertical, symbol Connector_Generic:Conn_02x05_Odd_Even
- J2: value CLOCK_IN -> STEP_IN
Connections:
- net +12V: now also J1.10 (Pin_10), J1.9 (Pin_9)
- net -12V: now also J1.1 (Pin_1), J1.2 (Pin_2)
- net GND: now also J1.3 (Pin_3), J1.4 (Pin_4), J1.5 (Pin_5), J1.6 (Pin_6), J1.7 (Pin_7), J1.8 (Pin_8)
Other:
- moved on the sheet: C7, C8, U3C
