File: Sequencer/Sequencer.kicad_pcb (KiCad board)
At the start: 2 copper layers, 125.7 x 99.1 mm, 116 parts, among them J1 CLOCK_IN, J2 RESET_IN, J3 FLIP_IN, J4 CV1_OUT, J5 CV2_OUT, J6 EURO_PWR_2x5, Q1 2N3904, Q2 2N3904, Q3 2N3904, SW1 SW_STEP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

Commit message: Sequencer progress
Parts:
- removed R1, R10, R11, R12, R13, R14, R15, R16, R2, R3, R4, R5, R6, R7, R8, R9: 100K, Resistor_THT:R_Axial_DIN0207_L6.3mm_D2.5mm_P2.54mm_Vertical
- added D15: 1N4148, Diode_THT:D_DO-35_SOD27_P7.62mm_Horizontal, F.Cu at (34.9, 43.8)
- added D16: 1N4148, Diode_THT:D_DO-35_SOD27_P7.62mm_Horizontal, F.Cu at (52.1, 43.8)
- added D17: 1N4148, Diode_THT:D_DO-35_SOD27_P7.62mm_Horizontal, F.Cu at (69.2, 43.8)
- added D18: 1N4148, Diode_THT:D_DO-35_SOD27_P7.62mm_Horizontal, F.Cu at (86.4, 43.8)
- added D19: 1N4148, Diode_THT:D_DO-35_SOD27_P7.62mm_Horizontal, F.Cu at (103.5, 43.8)
- added D20: 1N4148, Diode_THT:D_DO-35_SOD27_P7.62mm_Horizontal, F.Cu at (120.7, 43.8)
- added D21: 1N4148, Diode_THT:D_DO-35_SOD27_P7.62mm_Horizontal, F.Cu at (137.8, 43.8)
- added D22: 1N4148, Diode_THT:D_DO-35_SOD27_P7.62mm_Horizontal, F.Cu at (154.9, 43.8)
- added D23: 1N4148, Diode_THT:D_DO-35_SOD27_P7.62mm_Horizontal, F.Cu at (36.8, 64.1)
- added D24: 1N4148, Diode_THT:D_DO-35_SOD27_P7.62mm_Horizontal, F.Cu at (54.0, 64.1)
- added D25: 1N4148, Diode_THT:D_DO-35_SOD27_P7.62mm_Horizontal, F.Cu at (71.1, 64.1)
- added D26: 1N4148, Diode_THT:D_DO-35_SOD27_P7.62mm_Horizontal, F.Cu at (88.3, 64.1)
- added D27: 1N4148, Diode_THT:D_DO-35_SOD27_P7.62mm_Horizontal, F.Cu at (105.4, 64.1)
- added D28: 1N4148, Diode_THT:D_DO-35_SOD27_P7.62mm_Horizontal, F.Cu at (122.6, 64.1)
- added D29: 1N4148, Diode_THT:D_DO-35_SOD27_P7.62mm_Horizontal, F.Cu at (139.7, 64.1)
- added D30: 1N4148, Diode_THT:D_DO-35_SOD27_P7.62mm_Horizontal, F.Cu at (156.8, 63.5)
- J6: value EURO_PWR_2x5 -> Power; moved to F.Cu
- moved R57 273.8 mm to (144.8, 85.7)
- moved R56 270.6 mm to (150.9, 81.9)
- moved R55 269.0 mm to (148.8, 85.7), turned to 0 degrees
- moved R58 265.1 mm to (136.6, 85.7), turned to 0 degrees
- moved R59 260.6 mm to (132.6, 85.7)
- moved R53 256.4 mm to (136.6, 70.6), turned to 0 degrees
- moved R60 253.7 mm to (126.1, 85.7)
- moved R52 250.5 mm to (130.5, 70.6), turned to 0 degrees
- moved R61 247.1 mm to (120.0, 85.7), turned to -90 degrees
- moved R51 246.8 mm to (126.5, 70.6)
- moved R50 239.1 mm to (118.4, 70.6), turned to 0 degrees
- moved R49 235.8 mm to (114.7, 70.5)
- moved R54 235.5 mm to (114.9, 85.7), turned to -90 degrees
- moved C3 227.9 mm to (85.3, 91.4), turned to 90 degrees
- moved R48 226.0 mm to (112.6, 74.3), turned to 0 degrees
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Connections:
- J6 pad 1: +12V -> -12V
- J6 pad 10: -12V -> +12V
- J6 pad 2: +12V -> -12V
- J6 pad 9: -12V -> +12V
- R59 pad 2: Net-(U2D-+) -> Net-(U2D--)
- R60 pad 1: Net-(U2D-+) -> Net-(U2D--)
- U1 pad 21: STEP9 -> STEP16
- U1 pad 22: STEP10 -> STEP15
- U1 pad 23: STEP11 -> STEP14
- U1 pad 24: STEP12 -> STEP13
- U1 pad 25: STEP13 -> STEP12
- U1 pad 26: STEP14 -> STEP11
- U1 pad 27: STEP15 -> STEP10
- U1 pad 28: STEP16 -> STEP9
- U2 pad 10: CV2_OUT -> GND
- U2 pad 12: Net-(U2D-+) -> GND
- U2 pad 13: GND -> Net-(U2D--)
- U2 pad 9: GND -> CV2_OUT
Routing:
- net CV1_OUT: track 0.00 -> 234.2 mm
- net Net-(D23-K): track 0.00 -> 210.7 mm
- net +5V: track 0.00 -> 201.9 mm
- net -12V: track 0.00 -> 127.3 mm
- net STEP16: track 0.00 -> 85.7 mm
- net STEP8: track 0.00 -> 81.7 mm
- net STEP15: track 0.00 -> 72.3 mm
- net STEP7: track 0.00 -> 70.2 mm
- net STEP9: track 0.00 -> 70.1 mm
- net +12V: track 0.00 -> 69.0 mm
- net STEP1: track 0.00 -> 66.5 mm
- net Net-(D11-K): track 0.00 -> 63.3 mm
- net Net-(D12-K): track 0.00 -> 63.3 mm
- net Net-(D14-K): track 0.00 -> 62.6 mm
- net STEP6: track 0.00 -> 60.4 mm
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- added copper zone on B.Cu, net GND
- added copper zone on F.Cu, net GND
Other:
- board size 125.7 x 99.1 mm -> 139.7 x 99.1 mm
